Commit message: last working version

File: resource/urdf/obj_libs/trashbins/t2/model.urdf (robot description, URDF)
Before this commit: robot model.urdf, 1 links, 0 joints
Links:
- link model: geometry collision mesh filename=model_normalized_v.obj scale=1.5 1 1.5; visual mesh filename=model_normalized_v.obj scale=1.5 1 1.5
